File: week02/day00/ex00/propro/File: led.kicad_sch (KiCad schematic)
At the start: 2 parts

Commit message: add pcd + footprint lib
Parts:
- renumbered D1 to D4, R3 to R6
Connections:
- net GND: now also R6.2; no longer R6.
- net input: now also D4.1; no longer D4.
- new net: D4.2, R6.1
Changed lines of the file:
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@@
   (symbol (lib_id "Mylib:resistance") (at 44.958 34.036 0)
     (in_bom yes) (on_board yes)
-    (property "Reference" "R3" (id 0) (at 44.8564 31.2674 0)
+    (property "Reference" "R6" (id 0) (at 44.8564 31.2674 0)
       (effects (font (size 0.9 0.9)))
     )
@@
       (effects (font (size 1.27 1.27)) hide)
     )
-    (pin "")
-    (pin "")
+    (pin "1")
+    (pin "2")
   )
   (symbol (lib_id "Mylib:LED") (at 36.6522 34.0868 0)
     (in_bom yes) (on_board yes)
-    (property "Reference" "D1" (id 0) (at 35.3314 31.75 0))
+    (property "Reference" "D4" (id 0) (at 35.3314 31.75 0))
     (property "Value" "LED" (id 1) (at 38.3286 31.6992 0))
     (property "Footprint" "Footprint_lib:Led" (id 2) (at 36.6522 34.0868 0)
@@
       (effects (font (size 1.27 1.27)) hide)
     )
-    (pin "")
-    (pin "")
+    (pin "1")
+    (pin "2")
   )
   (symbol (lib_id "power:GND") (at 49.6316 35.814 0)
