File: week02/day00/ex00/propro/_autosave-File: usb_flasher.kicad_sch (KiCad schematic)
At the start: 2 parts, among them J1 Conn_01x86

Commit message: add pcd + footprint lib
Connections:
- net reset: now also C3.2; no longer C3.
- net at J1.5: now also C3.1; no longer C3.
Changed lines of the file:
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@@
       (effects (font (size 1.27 1.27)) hide)
     )
-    (pin "")
-    (pin "")
+    (pin "1")
+    (pin "2")
   )
   (symbol (lib_id "Mylib:Connector") (at 34.6456 29.5402 0) (unit 1)
