File: week02/day00/ex00/propro/button.kicad_sch (KiCad schematic)
At the start: 2 parts, among them SW1 SW_PUSH

Commit message: add pcd + footprint lib
Parts:
- R1: footprint (none) -> Footprint_lib:resistence
- SW1: footprint (none) -> Footprint_lib:sw
Connections:
- net +5V: now also R1.2; no longer R1.
- net GND: now also SW1.2; no longer SW1.
- net out: now also R1.1, SW1.1; no longer R1., SW1.
Changed lines of the file:
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@@
       (effects (font (size 0.8 0.8)) (justify right))
     )
-    (property "Footprint" "" (id 2) (at 47.498 43.434 0)
+    (property "Footprint" "Footprint_lib:resistence" (id 2) (at 47.498 43.434 0)
       (effects (font (size 1.27 1.27)) hide)
     )
@@
       (effects (font (size 1.27 1.27)) hide)
     )
-    (pin "")
-    (pin "")
+    (pin "1")
+    (pin "2")
   )
   (symbol (lib_id "power:GND") (at 47.5488 52.7812 0)
@@
       (effects (font (size 0.7 0.7)) (justify left))
     )
-    (property "Footprint" "" (id 2) (at 47.5488 50.4444 0)
+    (property "Footprint" "Footprint_lib:sw" (id 2) (at 47.5488 50.4444 0)
       (effects (font (size 1.27 1.27)) hide)
     )
@@
       (effects (font (size 1.27 1.27)) hide)
     )
-    (pin "")
-    (pin "")
+    (pin "1")
+    (pin "2")
   )
   (symbol (lib_id "power:+5V") (at 47.498 40.64 0)
