File: week02/day00/ex00/propro/propro.kicad_pcb (KiCad board)
At the start: 2 copper layers, 29 x 21.1 mm, 22 parts, among them J1 Conn_01x86, J2 AVR-ISP, SW1 SW_PUSH, SW2 SW_PUSH, U1 Atmega328p, Y1 16MHz

Commit message: add pcd + footprint lib
Parts:
- moved D1 0.37 mm to (103.5, 45.9)
- moved D4 0.28 mm to (103.5, 40.7)
- moved D2 0.20 mm to (103.5, 44.2)
- moved D3 0.08 mm to (103.5, 42.4)
Routing:
- net +5V: track 59.2 -> 65.6 mm, vias 1 -> 4
- net /~{RESET}: track 61.1 -> 60.4 mm
- net GND: track 106.1 -> 105.6 mm
- net /MISO: track 6.85 -> 6.95 mm, vias 1 -> 2
- net /SCK: track 10.8 -> 10.7 mm, vias 0 -> 1
- added copper zone on B.Cu, net GND
- added copper zone on F.Cu, net GND
