File: week02/day00/ex00/propro/propro.kicad_sch (KiCad schematic)
At the start: 8 parts, among them J2 AVR-ISP, U1 Atmega328p, Y1 16MHz

Commit message: add pcd + footprint lib
Connections:
- net +5V: now also C4.2, C5.2; no longer C4., C5.
- net GND: now also C1.1, C2.1, C4.1, C5.1; no longer C1., C2., C4., C5.
- net at U1.8 (XTAL2/PB7), Y1.1: now also C1.2; no longer C1.
- net at U1.7 (XTAL1/PB6), Y1.3: now also C2.2; no longer C2.
Changed lines of the file:
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@@
 (kicad_sch (version 20211123) (generator eeschema)
   (paper "A4")
+  (bus_alias "uart_buts" (members "~{RESET}" "MCU_RX" "MCU_TX" "BUT_0"))
   (bus_alias "LED" (members "LED_0" "LED_1" "LED_2" "LED_3_MOSI"))
-  (bus_alias "uart_buts" (members "~{RESET}" "MCU_RX" "MCU_TX" "BUT_0"))
   (junction (at 37.084 38.608) (diameter 0) (color 0 0 0 0)
   )
@@
       (effects (font (size 1.27 1.27)) hide)
     )
-    (pin "")
-    (pin "")
+    (pin "1")
+    (pin "2")
   )
   (symbol (lib_id "Mylib:mountingHole") (at 91.186 53.1876 0) (unit 1)
@@
       (effects (font (size 1.27 1.27)) hide)
     )
-    (pin "")
-    (pin "")
+    (pin "1")
+    (pin "2")
   )
   (symbol (lib_id "power:GND") (at 48.26 31.75 0) (unit 1)
@@
       (effects (font (size 1.27 1.27)) hide)
     )
-    (pin "")
-    (pin "")
+    (pin "1")
+    (pin "2")
   )
   (symbol (lib_id "power:GND") (at 50.1904 52.07 0) (unit 1)
@@
       (effects (font (size 1.27 1.27)) hide)
     )
-    (pin "")
-    (pin "")
+    (pin "1")
+    (pin "2")
   )
   (symbol (lib_id "power:PWR_FLAG") (at 84.3788 50.1142 0) (unit 1)
